File: PCB/Remote_RX:TX/RX/RC_Transmitter_RX_v42.sch (EAGLE design)
At the start: 27 parts, among them IC1 LAMBDA80C-24S, IC4 ESP32-WROVER-IE-N16R8, J1 MOLEX_53261-0271MOLEX_53261-0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, SW1 KMR2, SW2 KMR2, U1 AP2112K-3.3TRG1SOT_RG1_DIO-L, U2 AP2112K-3.3TRG1SOT_RG1_DIO-L

Commit message: Remote RX - PCB Update
Connections:
- net 3.3V: no longer R6.1
- net VIN: now also R6.1
Changed lines of the file:
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@@
 <part name="R6" library="SparkFun-Resistors" library_urn="urn:adsk.eagle:library:532" deviceset="0OHM" device="-0603-1/10W-5%" package3d_urn="urn:adsk.eagle:package:39650/1" value="10k"/>
 <part name="GND10" library="supply1" library_urn="urn:adsk.eagle:library:371" deviceset="GND" device=""/>
-<part name="U$7" library="microbuilder" deviceset="3.3V" device=""/>
 <part name="LS1" library="SMTB-0940-T-3V-R" deviceset="SMTB-0940-T-3V-R" device=""/>
 <part name="GND13" library="supply1" library_urn="urn:adsk.eagle:library:371" deviceset="GND" device=""/>
@@
 <part name="R9" library="SparkFun-Resistors" library_urn="urn:adsk.eagle:library:532" deviceset="0OHM" device="-0603-1/10W-5%" package3d_urn="urn:adsk.eagle:package:39650/1" value="0"/>
 <part name="U$2" library="microbuilder" deviceset="3.3V" device=""/>
+<part name="U$7" library="microbuilder" deviceset="VIN" device=""/>
 </parts>
 <sheets>
@@
 <attribute name="VALUE" x="-30.56" y="77.74" size="1.778" layer="96" rot="R270"/>
 </instance>
-<instance part="U$7" gate="G$1" x="-27.94" y="48.26" smashed="yes" rot="R90">
-<attribute name="VALUE" x="-28.956" y="46.736" size="1.27" layer="96" rot="R90"/>
-</instance>
 <instance part="LS1" gate="G$1" x="45.72" y="157.48" smashed="yes">
 <attribute name="NAME" x="44.45" y="163.83" size="1.778" layer="95"/>
@@
 <instance part="U$2" gate="G$1" x="15.24" y="142.24" smashed="yes">
 <attribute name="VALUE" x="13.716" y="143.256" size="1.27" layer="96"/>
+</instance>
+<instance part="U$7" gate="G$1" x="-27.94" y="48.26" smashed="yes" rot="R90">
+<attribute name="VALUE" x="-28.956" y="46.736" size="1.27" layer="96" rot="R90"/>
 </instance>
 </instances>
@@
 </segment>
 <segment>
-<pinref part="U$7" gate="G$1" pin="3.3V"/>
-<wire x1="-25.4" y1="48.26" x2="-25.4" y2="50.8" width="0.1524" layer="91"/>
-<pinref part="R6" gate="G$1" pin="1"/>
-</segment>
-<segment>
 <pinref part="R7" gate="G$1" pin="2"/>
 <wire x1="10.16" y1="137.16" x2="10.16" y2="139.7" width="0.1524" layer="91"/>
@@
 <junction x="7.62" y="0"/>
 </segment>
+<segment>
+<wire x1="-25.4" y1="48.26" x2="-25.4" y2="50.8" width="0.1524" layer="91"/>
+<pinref part="R6" gate="G$1" pin="1"/>
+<pinref part="U$7" gate="G$1" pin="VIN"/>
+</segment>
 </net>
 <net name="GPIO35*" class="0">
@@
 <wire x1="-81.28" y1="185.42" x2="-93.98" y2="185.42" width="0.1524" layer="91"/>
 <label x="-93.98" y="185.42" size="1.778" layer="95"/>
-</segment>
-<segment>
+<label x="-22.86" y="60.96" size="1.778" layer="95"/>
+</segment>
+<segment>
