File: PCB/Remote_RX:TX/RX/RC_Transmitter_RX_FINAL_v4.4.brd (EAGLE design)
At the start: 50 x 70 mm, 27 parts, among them IC1 LAMBDA80C-24S, IC4 ESP32-WROVER-IE-N16R8, J1 MOLEX_53261-0271MOLEX_53261-0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, SW1 KMR2, SW2 KMR2, U1 AP2112K-3.3TRG1SOT_RG1_DIO-L, U2 AP2112K-3.3TRG1SOT_RG1_DIO-L

Commit message: PCB Update
Parts:
- removed LS1: SMTB-0940-T-3V-R, SMTB-0940-T-3V-R:XDCR_SMTB-0940-T-3V-R
- removed R2: 0, SparkFun-Resistors:0603
- added BZ1: PKMCS0909E4000-R1, Microphone:PKMCS0909E4000-R1
- added C10, C12, C13, C14, C15: 10uF, SparkFun-Capacitors:0805
- added C11, C3, C4: 0.1uF, SparkFun-Capacitors:0805
- added C16, C17: 1.0uF, SparkFun-Capacitors:0805
- added C9: 6.2 pF, Capacitor:CAPC2012X110
- added J2: MOLEX_53261-0271MOLEX_53261-0271_0_0, Molex - 53261-0271:MOLEX_53261-0271_0
- C1, C2: value 10uF -> 0.1uF
- C7: value 6.2 pF -> 0.1uF; device Capacitor:CAPC2012X110 -> SparkFun-Capacitors:0805
- R1: value 0 -> 10k
- R3: value 56.2 kOhms -> 10M
- moved C7 52.4 mm to (34.4, 61.9), flipped to the bottom, turned to 180 degrees
- moved C6 32.6 mm to (34.4, 64.1), flipped to the bottom
- moved R1 32.0 mm to (11.1, 47.2), turned to 0 degrees
- moved C2 8.62 mm to (7.76, 52.9)
- moved C8 5.54 mm to (30.8, 14.4)
- moved C1 4.66 mm to (7.54, 61.8), flipped to the bottom, turned to 0 degrees
- moved CRYSTAL 4.01 mm to (32.2, 19.2)
- moved R3 3.50 mm to (31.9, 22.6)
- moved U1 1.16 mm to (12.9, 57.8)
- moved U2 1.12 mm to (7.82, 57.8)
- moved R4 1.10 mm to (9.01, 17.7)
- renumbered SW1 to RST, SW2 to GPIO0
Connections:
- removed net N$2: C8.2, CRYSTAL.2, R2.1, R3.1
- net 3.3V: now also C14.1, C16.2, C17.2, C2.1, C7.1
- net 3.3V*: now also C10.1, C11.1, C15.1, C4.1
- net GND: now also BZ1.2, C10.2, C11.2, C12.2, C13.2, C14.2, C15.2, C16.1, C17.1, C3.2, C4.2, C7.2, C9.1, J2.2, J2.3, J2.4; no longer C7.1, LS1.N
- net GPIO12(HMISO): now also J2.1
- net GPIO22: now also R1.2; no longer LS1.P
- net GPIO32*: now also C8.2, CRYSTAL.1, R3.2; no longer R1.2
- net GPIO33*: now also C9.2, CRYSTAL.2, R3.1; no longer R2.2
- net N$1: now also BZ1.1; no longer C7.2, CRYSTAL.1, R3.2
- net VIN: now also C12.1, C13.1, C3.1; no longer C2.1
Routing:
- net GPIO12(HMISO): track 0.00 -> 43.1 mm, vias 0 -> 4
- net GND: track 44.3 -> 14.0 mm, vias 6 -> 5
- net N$2: track 11.4 -> 0.00 mm
- net GPIO33*: track 2.84 -> 11.1 mm
- net GPIO32*: track 3.27 -> 11.1 mm
- net VIN: track 54.0 -> 61.7 mm, vias 2 -> 6
- net N$1: track 11.1 -> 5.31 mm
- net GPIO4*: track 39.3 -> 34.4 mm
- net 3.3V: track 146.4 -> 141.8 mm, vias 2 -> 4
- net GPIO26*: track 53.4 -> 48.8 mm
- net GPIO22: track 20.9 -> 16.8 mm
- net GPIO15*: track 34.2 -> 30.9 mm
- net GPIO25*: track 21.3 -> 18.4 mm
- net GPIO27*: track 17.8 -> 16.1 mm
- net GPIO0: track 55.8 -> 54.2 mm
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Other:
- board text added: "v4.4"
- board text removed: "v4.2"
