File: PCB/Remote_RX:TX/RX/RC_Transmitter_RX_FINAL_v4.4.sch (EAGLE design)
At the start: 37 parts, among them IC1 LAMBDA80C-24S, IC2 MCP23S17T-E_ML, IC3 MCP23S17T-E_ML, IC4 ESP32-WROVER-IE-N16R8, IC5 MCP3208-CI_SL, IC6 MCP3208-CI_SL, J1 MOLEX_53261-0271MOLEX_53261-0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, SW1 KMR2, SW2 KMR2, U1 AP2112K-3.3TRG1SOT_RG1_DIO-L, U2 AP2112K-3.3TRG1SOT_RG1_DIO-L

Commit message: PCB Update
Parts:
- removed ANO_1, ANO_2: 0532610871, 0532610871:0532610871
- removed IC2, IC3: MCP23S17T-E_ML, MCP23S17T-E_ML:MCP23S17T-E_ML
- removed IC5, IC6: MCP3208-CI_SL, MCP3208-CI_SL:MCP3208-CI_SL
- removed JOYSTICK1, JOYSTICK2, POT_SIG_2, SWITCHES: 0532610671, 0532610671:0532610671
- removed POT_SIG_1: 0532611071, 0532611071:0532611071
- removed R2: 0, SparkFun-Resistors:0OHM-0603-1/10W-5%
- added BZ1: PKMCS0909E4000-R1, Microphone:PKMCS0909E4000-R1
- added C12, C13, C14, C15: 10uF, SparkFun-Capacitors:10UF-0805-10V-10%
- added C16, C17: 1.0uF, SparkFun-Capacitors:10UF-0805-10V-10%
- added J2: MOLEX_53261-0271MOLEX_53261-0271_0_0, Molex - 53261-0271:MOLEX_53261-0271MOLEX_53261-0271_0_0
- added LCD: 0532610871, 0532610871:0532610871
- added PUSH_BUTTONS: 0532610471, 0532610471:0532610471
- added R7, R8, R9: 0, SparkFun-Resistors:0OHM-0603-1/10W-5%
- C1, C2, C3: value 10uF -> 0.1uF
- C10: value 0.1uF -> 10uF
- C5: value 0.1uF -> 1uF; device SparkFun-Capacitors:10UF-0805-10V-10% -> microbuilder:CAP_CERAMIC0805-NOOUTLINE
- C7: value 6.2 pF -> 0.1uF; device Capacitor:C_CHIP-0805(2012-METRIC) -> SparkFun-Capacitors:10UF-0805-10V-10%
- C9: value 1uF -> 6.2 pF; device microbuilder:CAP_CERAMIC0805-NOOUTLINE -> Capacitor:C_CHIP-0805(2012-METRIC)
- R1: value 0 -> 10k
- R3: value 56.2 kOhms -> 10M
- R5, R6: value 10K -> 10k; device microbuilder:RESISTOR_0805 -> SparkFun-Resistors:0OHM-0603-1/10W-5%
- renumbered SW1 to RST, SW2 to GPIO0
Connections:
- removed net ANO1_ENCA: ANO_1.8, IC2.GPB7
- removed net ANO1_ENCB: ANO_1.7, IC2.GPB6
- removed net ANO1_SW1: ANO_1.6, IC2.GPB5
- removed net ANO1_SW2: ANO_1.5, IC2.GPB4
- removed net ANO1_SW3: ANO_1.4, IC2.GPB3
- removed net ANO1_SW4: ANO_1.3, IC2.GPB2
- removed net ANO1_SW5: ANO_1.2, IC2.GPB1
- removed net ANO2_ENCA: ANO_2.8, IC2.GPA7
- removed net ANO2_ENCB: ANO_2.7, IC2.GPA6
- removed net ANO2_SW1: ANO_2.6, IC2.GPA5
- removed net ANO2_SW2: ANO_2.5, IC2.GPA4
- removed net ANO2_SW3: ANO_2.4, IC2.GPA3
- removed net ANO2_SW4: ANO_2.3, IC2.GPA2
- removed net ANO2_SW5: ANO_2.2, IC2.GPA1
- removed net GPIO15: IC4.IO15
- removed net GPIO22*: IC3.!CS, IC4.IO22
- removed net GPIO34: IC4.IO34
- removed net GPIO35: IC4.IO35
- removed net GPIO36: IC4.SENSOR_VP
- removed net GPIO39: IC4.SENSOR_VN
- removed net JOYSTICK_X1: IC6.CH0, JOYSTICK1.3
- removed net JOYSTICK_X2: IC6.CH2, JOYSTICK2.3
- removed net JOYSTICK_Y1: IC6.CH1, JOYSTICK1.6
- removed net JOYSTICK_Y2: IC6.CH3, JOYSTICK2.6
- removed net N$10: IC5.CH7
- removed net N$2: C8.2, CRYSTAL.X2, R2.1, R3.1
- removed net N$4: IC2.!RESET, R5.2
- removed net N$5: IC3.!RESET, R6.2
- removed net N$9: IC5.CH6
- removed net POT1: IC5.CH0, POT_SIG_1.6
- removed net POT1_SW: IC3.GPA0, POT_SIG_1.7
- removed net POT2: IC5.CH1, POT_SIG_1.5
- removed net POT2_SW: IC3.GPA1, POT_SIG_1.8
- removed net POT3: IC5.CH2, POT_SIG_1.4
- removed net POT3_SW: IC3.GPA2, POT_SIG_1.9
- removed net POT4: IC5.CH3, POT_SIG_1.3
- removed net POT4_SW: IC3.GPA3, POT_SIG_1.10
- removed net POT5: IC5.CH4, POT_SIG_2.3
- removed net POT5_SW: IC3.GPA4, POT_SIG_2.4
- removed net POT6: IC5.CH5, POT_SIG_2.5
- removed net POT6_SW: IC3.GPA5, POT_SIG_2.6
- removed net SW1: IC3.GPB0, SWITCHES.2
- removed net SW2: IC3.GPB1, SWITCHES.3
- removed net SW3: IC3.GPB2, SWITCHES.4
- removed net SW4: IC3.GPB3, SWITCHES.5
- removed net SW5: IC3.GPB4, SWITCHES.6
- new net GPIO15*: IC4.IO15, LCD.8
- new net GPIO22: IC4.IO22, R1.2
- new net GPIO34*: IC4.IO34, PUSH_BUTTONS.4, R9.1
- new net GPIO35*: IC4.IO35, R5.1, R6.2
- new net GPIO36*: IC4.SENSOR_VP, PUSH_BUTTONS.2, R7.1
- new net GPIO39*: IC4.SENSOR_VN, PUSH_BUTTONS.3, R8.1
- net 3.3V: now also C14.1, C16.2, C17.2, C2.1, C7.1, LCD.2, R7.2, R8.2, R9.2; no longer C10.2, C11.2, C2.2, C3.2, C4.2, C5.2, IC2.VDD, IC3.A2, IC3.VDD, IC5.VDD, IC5.VREF, IC6.VDD, IC6.VREF, JOYSTICK1.2, JOYSTICK1.5, JOYSTICK2.2, JOYSTICK2.5, POT_SIG_1.2, POT_SIG_2.2, R5.1, R6.1
- net 3.3V*: now also C10.1, C11.1, C15.1, C4.1
- net GND: now also BZ1.2, C10.2, C11.2, C12.2, C13.2, C14.2, C15.2, C16.1, C17.1, C2.2, C3.2, C4.2, C5.2, C7.2, C9.1, J2.2, J2.MNT_1, J2.MNT_2, LCD.1, PUSH_BUTTONS.1, PUSH_BUTTONS.MP1, PUSH_BUTTONS.MP2, R5.2; no longer ANO_1.1, ANO_2.1, C10.1, C11.1, C2.1, C3.1, C4.1, C5.1, C7.1, C9.2, IC2.A0, IC2.A1, IC2.A2, IC2.VSS, IC3.A0, IC3.A1, IC3.VSS, IC5.AGND, IC5.DGND, IC6.AGND, IC6.DGND, JOYSTICK1.1, JOYSTICK1.4, JOYSTICK2.1, JOYSTICK2.4, POT_SIG_1.1, POT_SIG_1.MP1, POT_SIG_1.MP2, POT_SIG_2.1, SWITCHES.1
- net GPIO12(HMISO): now also J2.1; no longer IC2.SO, IC3.SO, IC5.DOUT, IC6.DOUT
- net GPIO13(HMOSI): now also LCD.6; no longer IC2.SI, IC3.SI, IC5.DIN, IC6.DIN
- net GPIO14(HSCLK): now also LCD.5; no longer IC2.SCK, IC3.SCK, IC5.CLK, IC6.CLK
- net GPIO25*: now also LCD.3; no longer IC5.!CS!/SHDN
- net GPIO27*: now also LCD.4; no longer IC6.!CS!/SHDN
- net GPIO32*: now also C8.2, CRYSTAL.X1, R3.2; no longer R1.2
- net GPIO33*: now also C9.2, CRYSTAL.X2, R3.1; no longer R2.2
- net GPIO4*: now also LCD.7; no longer IC2.!CS
- net N$1: now also BZ1.1; no longer C7.2, CRYSTAL.X1, R3.2
- net RST: now also C5.1; no longer C9.1
- net VIN: now also C12.1, C13.1, C3.1, R6.1
Other:
- note added: "Voltage Divider"
- moved on the sheet: C10, C11, C2, C3, C4, C5, C6, C7, C8, C9, R1, U1
