File: PCB/Remote_RX:TX/TX/RC_Transmitter_TX_FINAL_v4.4.sch (EAGLE design)
At the start: 27 parts, among them IC1 LAMBDA80C-24S, IC4 ESP32-WROVER-IE-N16R8, J1 MOLEX_53261-0271MOLEX_53261-0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, SW1 KMR2, SW2 KMR2, U1 AP2112K-3.3TRG1SOT_RG1_DIO-L, U2 AP2112K-3.3TRG1SOT_RG1_DIO-L

Commit message: PCB Update
Parts:
- removed LCD: 0532610871, 0532610871:0532610871
- removed LS1: SMTB-0940-T-3V-R, SMTB-0940-T-3V-R:SMTB-0940-T-3V-R
- removed PUSH_BUTTONS: 0532610471, 0532610471:0532610471
- removed R7, R8, R9: 0, SparkFun-Resistors:0OHM-0603-1/10W-5%
- added C10, C12, C13, C15, C17, C19, C21, C22, C23, C24, C28, C30, C32, C34, C37, C39: 0.1uF, SparkFun-Capacitors:10UF-0805-10V-10%
- added C11, C14, C16, C18, C20, C29, C3, C31, C33, C35, C36, C38, C4, C9: 10uF, SparkFun-Capacitors:10UF-0805-10V-10%
- added C25: 1uF, SparkFun-Capacitors:10UF-0805-10V-10%
- added C26, C27: 6.2 pF, SparkFun-Capacitors:10UF-0805-10V-10%
- added ENCODER_1, ENCODER_2: 0532610871, 0532610871:0532610871
- added IC2, IC3: MCP23S17T-E_ML, MCP23S17T-E_ML:MCP23S17T-E_ML
- added IC5, IC6: MCP3208-CI_SL, MCP3208-CI_SL:MCP3208-CI_SL
- added IN/OUT, JOYSTICK1, JOYSTICK2, POT_SIG_2, SWITCHES: 0532610671, 0532610671:0532610671
- added POT_SIG_1: 0532611071, 0532611071:0532611071
- C5: value 1uF -> 10uF; device microbuilder:CAP_CERAMIC0805-NOOUTLINE -> SparkFun-Capacitors:10UF-0805-10V-10%
- C6: value 10uF -> 0.1uF
- C7: value 6.2 pF -> 10uF; device Capacitor:C_CHIP-0805(2012-METRIC) -> SparkFun-Capacitors:10UF-0805-10V-10%
- C8: value 6.2 pF -> 0.1uF; device Capacitor:C_CHIP-0805(2012-METRIC) -> SparkFun-Capacitors:10UF-0805-10V-10%
- R1, R2: value 0 -> 10k
- R3: value 56.2 kOhms -> 10M
- R4: value 10K -> 10k; device microbuilder:RESISTOR_0805 -> SparkFun-Resistors:0OHM-0603-1/10W-5%
- renumbered SW1 to RST, SW2 to GPIO0
Connections:
- removed net GPIO15*: IC4.IO15, LCD.8
- removed net GPIO22: IC4.IO22, LS1.P
- removed net GPIO34*: IC4.IO34, PUSH_BUTTONS.4, R9.1
- removed net GPIO35*: IC4.IO35, R5.1, R6.2
- removed net GPIO36*: IC4.SENSOR_VP, PUSH_BUTTONS.2, R7.1
- removed net GPIO39*: IC4.SENSOR_VN, PUSH_BUTTONS.3, R8.1
- removed net N$1: C7.2, CRYSTAL.X1, R1.1, R3.2
- removed net N$2: C8.2, CRYSTAL.X2, R2.1, R3.1
- new net ANO1_ENCA: ENCODER_1.8, IC2.GPB7
- new net ANO1_ENCB: ENCODER_1.7, IC2.GPB6
- new net ANO1_SW1: ENCODER_1.6, IC2.GPB5
- new net ANO1_SW2: ENCODER_1.5, IC2.GPB4
- new net ANO1_SW3: ENCODER_1.4, IC2.GPB3
- new net ANO1_SW4: ENCODER_1.3, IC2.GPB2
- new net ANO1_SW5: ENCODER_1.2, IC2.GPB1
- new net ANO2_ENCA: ENCODER_2.8, IC2.GPA7
- new net ANO2_ENCB: ENCODER_2.7, IC2.GPA6
- new net ANO2_SW1: ENCODER_2.6, IC2.GPA5
- new net ANO2_SW2: ENCODER_2.5, IC2.GPA4
- new net ANO2_SW3: ENCODER_2.4, IC2.GPA3
- new net ANO2_SW4: ENCODER_2.3, IC2.GPA2
- new net ANO2_SW5: ENCODER_2.2, IC2.GPA1
- new net GPIO15: IC4.IO15, IN/OUT.6
- new net GPIO22*: IC3.!CS, IC4.IO22
- new net GPIO34: IC4.IO34, IN/OUT.2, R2.1
- new net GPIO35: IC4.IO35, IN/OUT.3, R4.1
- new net GPIO36: IC4.SENSOR_VP, IN/OUT.4, R5.2
- new net GPIO39: IC4.SENSOR_VN, IN/OUT.5, R6.2
- new net JOYSTICK_X1: IC6.CH0, IC6.CH1, JOYSTICK1.3
- new net JOYSTICK_X2: IC6.CH4, IC6.CH5, JOYSTICK2.3
- new net JOYSTICK_Y1: IC6.CH2, IC6.CH3, JOYSTICK1.6
- new net JOYSTICK_Y2: IC6.CH6, IC6.CH7, JOYSTICK2.6
- new net N$10: IC5.CH7
- new net N$9: IC5.CH6
- new net POT1: IC5.CH0, POT_SIG_1.6
- new net POT1_SW: IC3.GPA0, POT_SIG_1.7
- new net POT2: IC5.CH1, POT_SIG_1.5
- new net POT2_SW: IC3.GPA1, POT_SIG_1.8
- new net POT3: IC5.CH2, POT_SIG_1.4
- new net POT3_SW: IC3.GPA2, POT_SIG_1.9
- new net POT4: IC5.CH3, POT_SIG_1.3
- new net POT4_SW: IC3.GPA3, POT_SIG_1.10
- new net POT5: IC5.CH4, POT_SIG_2.3
- new net POT5_SW: IC3.GPA4, POT_SIG_2.4
- new net POT6: IC5.CH5, POT_SIG_2.5
- new net POT6_SW: IC3.GPA5, POT_SIG_2.6
- new net SW1: IC3.GPB0, SWITCHES.2
- new net SW2: IC3.GPB1, SWITCHES.3
- new net SW3: IC3.GPB2, SWITCHES.4
- new net SW4: IC3.GPB3, SWITCHES.5
- new net SW5: IC3.GPB4, SWITCHES.6
- net 3.3V: now also C10.2, C11.2, C12.2, C13.2, C14.2, C15.2, C16.2, C17.2, C18.2, C19.2, C2.1, C20.2, C22.1, C28.1, C29.1, C30.1, C31.1, C32.1, C33.1, C34.1, C35.1, C36.1, C37.1, C38.2, C39.2, C7.1, C8.1, C9.2, IC2.!RESET, IC2.VDD, IC3.!RESET, IC3.A2, IC3.VDD, IC5.VDD, IC5.VREF, IC6.VDD, IC6.VREF, JOYSTICK1.2, JOYSTICK1.5, JOYSTICK2.2, JOYSTICK2.5, POT_SIG_1.2, POT_SIG_2.2, R1.1, R2.2, R5.1, R6.1; no longer C6.1, LCD.2, R7.2, R8.2, R9.2
- net 3.3V*: now also C24.1, C4.1, C5.2, C6.2
- net GND: now also C10.1, C11.1, C12.1, C13.1, C14.1, C15.1, C16.1, C17.1, C18.1, C19.1, C20.1, C21.2, C22.2, C23.2, C24.2, C25.1, C26.1, C27.1, C28.2, C29.2, C3.2, C30.2, C31.2, C32.2, C33.2, C34.2, C35.2, C36.2, C37.2, C38.1, C39.1, C4.2, C5.1, C6.1, C7.2, C8.2, C9.1, ENCODER_1.1, ENCODER_2.1, IC2.A0, IC2.A1, IC2.A2, IC2.VSS, IC3.A0, IC3.A1, IC3.VSS, IC5.AGND, IC5.DGND, IC6.AGND, IC6.DGND, IN/OUT.1, JOYSTICK1.1, JOYSTICK1.4, JOYSTICK2.1, JOYSTICK2.4, POT_SIG_1.1, POT_SIG_1.MP1, POT_SIG_1.MP2, POT_SIG_2.1, SWITCHES.1; no longer C5.2, C6.2, C7.1, C8.1, LCD.1, LS1.N, PUSH_BUTTONS.1, PUSH_BUTTONS.MP1, PUSH_BUTTONS.MP2, R5.2
- net GPIO12(HMISO): now also IC2.SO, IC3.SO, IC5.DOUT, IC6.DOUT
- net GPIO13(HMOSI): now also IC2.SI, IC3.SI, IC5.DIN, IC6.DIN; no longer LCD.6
- net GPIO14(HSCLK): now also IC2.SCK, IC3.SCK, IC5.CLK, IC6.CLK; no longer LCD.5
- net GPIO25*: now also IC5.!CS!/SHDN; no longer LCD.3
- net GPIO27*: now also IC6.!CS!/SHDN; no longer LCD.4
- net GPIO32*: now also C26.2, CRYSTAL.X1, R3.2; no longer R1.2
- net GPIO33*: now also C27.2, CRYSTAL.X2, R3.1; no longer R2.2
- net GPIO4*: now also IC2.!CS; no longer LCD.7
- net RST: now also C25.2, R1.2; no longer C5.1, R4.1
- net VIN: now also C21.1, C23.1, C3.1; no longer C2.1, R6.1
Other:
- note removed: "Voltage Divider"
- moved on the sheet: C1, C2, C5, C6, C7, C8, R1, R2, R5, R6, U1, U2
